File: lcd-transposer.kicad_pcb (KiCad board)
At the start: 2 copper layers, 0 parts

Commit message: v1.0a
Parts:
- added LOWER1, UPPER1: JLX12864G-086, LocalLibrary:JLX12864G, F.Cu at (148.9, 99.5)
Routing:
- net /CS: track 0.00 -> 46.7 mm, vias 0 -> 1
- net /RST: track 0.00 -> 45.3 mm, vias 0 -> 1
- net /RS: track 0.00 -> 43.7 mm, vias 0 -> 1
- net /SDA: track 0.00 -> 42.2 mm, vias 0 -> 1
- net /SCK: track 0.00 -> 40.8 mm, vias 0 -> 1
- net /VDD: track 0.00 -> 39.3 mm, vias 0 -> 1
- net /LEDA: track 0.00 -> 38.2 mm, vias 0 -> 1
- net /VSS: track 0.00 -> 37.8 mm, vias 0 -> 1
Other:
- board outline added: 44.5 x 44.5 mm
- board text added: "JLCJLCJLCJLC"
- board text added: "LCD Interposer"
- board text added: "mjd@afork.com"
- board text added: "v1.0a 9-Oct-2023"
